Commit message: fixed joint state publishing

File: neo_description_mp_500/ros/robot/air_wheel.xacro (robot description, xacro)
@@ -27,4 +27,5 @@
     <mesh filename="package://neo_description_mp_500/ros/meshes/air_wheel_260.stl"/>
    </geometry>
+   <material name="Black" />
   </visual>
   <collision>

File: neo_description_mp_500/ros/robot/mp_500_0_9_base.xacro (robot description, xacro)
@@ -23,5 +23,5 @@
                 <origin xyz="0 0 0" rpy="0 0 0" />
                 <geometry>
-                    <mesh filename="package://neo_description_mp_500/ros/meshes/mp_s500_topplate.stl"/>
+                    <mesh filename="package://neo_description_mp_500/ros/meshes/mp_500_topplate.stl"/>
                 </geometry>
               <material name="Blue" />
@@ -30,9 +30,9 @@
                 <origin xyz="0. 0. 0.15" rpy="0 0 0" />
                 <geometry>
-                    <mesh filename="package://neo_description_mp_500/ros/meshes/mp_s500_topplate.stl"/>
+                    <mesh filename="package://neo_description_mp_500/ros/meshes/mp_500_topplate.stl"/>
                 </geometry>
             </collision>
         </link>
-        <joint name="base_caster_support_joint" type="continuous">
+        <joint name="base_caster_support_joint" type="fixed">
             <origin xyz="-0.5 0 0.08" rpy="0 0 0" />
             <parent link="base_link" />
@@ -63,5 +63,5 @@
             </collision>
         </link>
-        <joint name="caster_wheel_joint" type="continuous">
+        <joint name="caster_wheel_joint" type="fixed">
             <origin xyz="0. 0 0.0" rpy="0 0 0" />
             <parent link="base_caster_support_link" />
@@ -101,8 +101,8 @@
         </gazebo>
         <!-- MACRO INSTANTIATION -->
-        <air_wheel_260 suffix="left" parent="base_link">
+        <air_wheel_260 suffix="left_wheel" parent="base">
             <origin xyz="0. 0.3 0.13" rpy="0 0 0" />
         </air_wheel_260>
-        <air_wheel_260 suffix="right" parent="base_link">
+        <air_wheel_260 suffix="right_wheel" parent="base">
             <origin xyz="0. -0.3 0.13" rpy="0 0 0" />
         </air_wheel_260>

File: neo_description_mp_500/ros/robot/mp_500_2_1_base.xacro (robot description, xacro)
@@ -34,5 +34,5 @@
             </collision>
         </link>
-        <joint name="base_caster_support_joint" type="continuous">
+        <joint name="base_caster_support_joint" type="fixed">
             <origin xyz="-0.5 0 0.08" rpy="0 0 0" />
             <parent link="base_link" />
@@ -63,5 +63,5 @@
             </collision>
         </link>
-        <joint name="caster_wheel_joint" type="continuous">
+        <joint name="caster_wheel_joint" type="fixed">
             <origin xyz="0. 0 0.0" rpy="0 0 0" />
             <parent link="base_caster_support_link" />
