Commit message: mpo 500 simulation

File: neo_description_mpo_500/ros/robot/mpo_500_1_0_base.xacro (robot description, xacro)
@@ -53,4 +53,37 @@
          <origin xyz="-0.39 0 0" rpy="0 0 3.14" />
        </sick_s300_laser_v0>
+        <gazebo>
+            <controller:mecanum_drive_plugin name="mecanum_drive_controller" plugin="libmecanum_plugin.so">
+                <alwaysOn>true</alwaysOn>
+                <update>100</update>
+                <updateRate>100.0</updateRate>
+                <frontLeftJoint>wheel_front_left_joint</frontLeftJoint>
+                <frontRightJoint>wheel_front_right_joint</frontRightJoint>
+                <backLeftJoint>wheel_back_left_joint</backLeftJoint>
+                <backRightJoint>wheel_back_right_joint</backRightJoint>
+                <robotWidth>0.27</robotWidth>
+                <robotLength>0.25</robotLength>
+                <wheelDiameter>0.26</wheelDiameter>
+                <torque>5</torque>
+                <interface:position name="position_iface_0"/>
+                <topicName>cmd_vel</topicName>
+            </controller:mecanum_drive_plugin>
+            <controller:gazebo_ros_p3d name="p3d_base_controller" plugin="libgazebo_ros_p3d.so">
+                <alwaysOn>true</alwaysOn>
+                <updateRate>100.0</updateRate>
+                <bodyName>base_link</bodyName>
+                <topicName>base_pose_ground_truth</topicName>
+                <gaussianNoise>0.01</gaussianNoise>
+                <frameName>map</frameName>
+                <xyzOffsets>0 0 0</xyzOffsets>
+                <rpyOffsets>0 0 0</rpyOffsets>
+                <interface:position name="p3d_base_position"/>
+            </controller:gazebo_ros_p3d>
+            <controller:gazebo_ros_controller_manager name="gazebo_ros_controller_manager" plugin="libgazebo_ros_controller_manager.so">
+                <alwaysOn>true</alwaysOn>
+                <updateRate>100.0</updateRate>
+                <interface:audio name="gazebo_ros_controller_manager_dummy_iface" />
+            </controller:gazebo_ros_controller_manager>
+        </gazebo>
     </macro>
 </robot>

File: neo_description_mpo_500/ros/robot/omni_wheel.xacro (robot description, xacro)
@@ -42,4 +42,9 @@
   <!--material>Erratic/White</material-->
  </gazebo>
+ <transmission type="pr2_mechanism_model/SimpleTransmission" name="${suffix}_trans">
+  <actuator name="${suffix}_motor" />
+  <joint name="${suffix}_joint" />
+  <mechanicalReduction>1.0</mechanicalReduction>
+ </transmission>
 </macro>
 </robot>
